Commit message: corrected urdf

File: src/my_bot/description/camera.xacro (robot description, xacro)
@@ -4,16 +4,16 @@
         <parent link="chassis"/>
         <child link="camera"/>
-        <origin xyz="0.305 0 0.08" rpy="0.0 0.0 0.0"/>
+        <origin xyz="0.16 0 0.07" rpy="0.0 0.0 0.0"/>
     </joint>
     <link name="camera">
         <visual>
             <geometry>
-                <box size="0.01 0.03 0.03"/>
+                <box size="0.025 0.086 0.03"/>
             </geometry>
-            <material name="red"/>
+            <material name="black"/>
         </visual>
         <collision>
             <geometry>
-                <box size="0.01 0.03 0.03"/>
+                <box size="0.086 0.025 0.03"/>
             </geometry>
         </collision>

File: src/my_bot/description/lidar.xacro (robot description, xacro)
@@ -4,5 +4,5 @@
         <parent link="chassis"/>
         <child link="lidar"/>
-        <origin xyz="0.1 0 0.175" rpy="0.0 0.0 0.0"/>
+        <origin xyz="0 0 0.07" rpy="0.0 0.0 0.0"/>
     </joint>
     <link name="lidar">

File: src/my_bot/description/robot.urdf.xacro (robot description, xacro)
@@ -6,5 +6,5 @@
     <xacro:include filename="lidar.xacro" />
     <xacro:include filename="camera.xacro" />
-    <!-- <xacro:include filename="ros2_control.xacro" /> -->
-    <xacro:include filename="ros2_control_real.xacro" />
+    <xacro:include filename="ros2_control.xacro" />
+    <!-- <xacro:include filename="ros2_control_real.xacro" /> -->
 </robot>

File: src/my_bot/description/robot_core.xacro (robot description, xacro)
@@ -12,18 +12,18 @@
         <parent link="base_link"/>
         <child link="chassis"/>
-        <origin xyz="-0.1 0.0 0"/>
+        <origin xyz="0.13 0.0 0.12"/>
     </joint>
     <link name="chassis">
         <visual>
-            <origin xyz="0.15 0.0 0.075"/>
+            <origin xyz="0 0.0 0"/>
             <geometry>
-                <box size="0.3 0.3 0.15"/>
+                <box size="0.34 0.18 0.12"/>
             </geometry>
             <material name="white"/>
         </visual>
         <collision>
-            <origin xyz="0.15 0.0 0.075"/>
+            <origin xyz="0.13 0.0 0.12"/>
             <geometry>
-                <box size="0.3 0.3 0.15"/>
+                <box size="0.34 0.18 0.12"/>
             </geometry>
         </collision>
@@ -39,5 +39,5 @@
         <parent link="base_link"/>
         <child link="left_wheel"/>
-        <origin xyz="0.0 0.175 0.0" rpy="-${pi/2} ${pi} 0.0"/>
+        <origin xyz="0.0 0.1 0.042" rpy="-${pi/2} ${pi} 0.0"/>
         <axis xyz="0.0 0.0 1"/>
      </joint>
@@ -45,5 +45,5 @@
         <visual>
             <geometry>
-                <cylinder radius="0.085" length="0.04"/>
+                <cylinder radius="0.042" length="0.04"/>
             </geometry>
             <material name="black"/>
@@ -51,5 +51,5 @@
         <collision>
             <geometry>
-                <cylinder radius="0.05" length="0.04"/>
+                <cylinder radius="0.042" length="0.04"/>
             </geometry>
         </collision>
@@ -65,5 +65,5 @@
         <parent link="base_link"/>
         <child link="right_wheel"/>
-        <origin xyz="0.0 -0.175 0.0" rpy="${pi/2} 0 0.0"/>
+        <origin xyz="0.0 -0.1 0.042" rpy="${pi/2} 0 0.0"/>
         <axis xyz="0.0 0.0 -1"/>
      </joint>
@@ -71,5 +71,5 @@
         <visual>
             <geometry>
-                <cylinder radius="0.085" length="0.04"/>
+                <cylinder radius="0.042" length="0.04"/>
             </geometry>
             <material name="black"/>
@@ -77,5 +77,5 @@
         <collision>
             <geometry>
-                <cylinder radius="0.05" length="0.04"/>
+                <cylinder radius="0.042" length="0.04"/>
             </geometry>
         </collision>
@@ -91,19 +91,19 @@
         <parent link="chassis"/>
         <child link="caster_wheel"/>
-        <origin xyz="0.24 0.0 0.0"/>
+        <origin xyz="0.13 0.0 -0.09"/>
      </joint>
      <link name="caster_wheel">
         <visual>
             <geometry>
-                <sphere radius="0.05"/>
+                <sphere radius="0.04"/>
             </geometry>
-            <material name="silver"/>
+            <material name="gold"/>
         </visual>
         <collision>
             <geometry>
-                <sphere radius="0.05"/>
+                <sphere radius="0.04"/>
             </geometry>
         </collision>
-        <xacro:inertial_sphere mass="0.1" radius="0.05">
+        <xacro:inertial_sphere mass="0.1" radius="0.04">
             <origin xyz="0.0 0.0 0.0" rpy="0.0 0.0 0.0"/>
         </xacro:inertial_sphere>

File: src/my_bot/description/ros2_control.xacro (robot description, xacro)
@@ -24,32 +24,7 @@
     <gazebo>
         <plugin filename="libgz_ros2_control-system.so" name="gz_ros2_control::GazeboSimROS2ControlPlugin">
-            <parameters>/home/jrm/dev_ws/src/my_bot/config/my_controllers.yaml</parameters>
+            <parameters>/home/jrm/spiader/src/my_bot/config/my_controllers.yaml</parameters>
             <controller_manager_prefix_node_name>controller_manager</controller_manager_prefix_node_name>
         </plugin>
     </gazebo>
-    <!-- <ros2_control name = "arduino_drive" type = "system">
-        <hardware>
-            <plugin>my_bot/MyBotArduinoHardware</plugin>
-            <param name="device">/dev/ttyACM0</param> <!--change this to the correct USB-->
-            <param name="baud_rate">115200</param>
-            <param name="timeout_ms">1000</param>
-            <param name="enc_counts_per_rev">330</param>
-        </hardware>
-        <joint name="left_wheel_joint">
-            <command_interface name="velocity">
-                <param name="min">-10</param>
-                <param name="max">10</param>
-            </command_interface>
-            <state_interface name = "velocity"/>
-            <state_interface name = "position"/>
-        </joint>
-        <joint name="right_wheel_joint">
-            <command_interface name="velocity">
-                <param name="min">-10</param>
-                <param name="max">10</param>
-            </command_interface>
-            <state_interface name = "velocity"/>
-            <state_interface name = "position"/>
-        </joint>
-    </ros2_control> -->
 </robot>
